File: KiCad/MDBT42STICK.sch (KiCad schematic (older format))
At the start: 28 parts, among them P1 CONN_01X04, P12 SERIALBUS, P2 USB_B, P3 CONN_01X07, P4 CONN_01X01, P5 CONN_01X03, P7 PROGRAM, SW1 RESET, U1 ADMP401Module, U2 MDBT42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

Commit message: 2nd version.
Parts:
- removed C10: 0.1μF, Capacitors_SMD:C_1206, symbol C
- removed C11: 1μF, Capacitors_SMD:C_1206, symbol C
- removed C9: 4.7μF, Capacitors_SMD:C_1206, symbol C
- removed P12: SERIALBUS, library:SolderWirePad_Circle_5xInline_0-8mmDrill, symbol CONN_01X05
- removed P2: USB_B, library:USB-4AM103, symbol USB_B
- removed P3: CONN_01X07, Pin_Headers:Pin_Header_Straight_1x07, symbol CONN_01X07
- removed P7: PROGRAM, library:SolderWirePad_Circle_5xInline_0-8mmDrill, symbol CONN_01X05
- removed U4: CP2104, library:QFN-24_HandSoldering, symbol CP2104
- removed U5: MPU-6500_Module, library:MPU-6500_GY-6500, symbol MPU-6500_Module
- added P2: CONN_01X08, library:SolderWirePad_Circle_8xInline_0-85mmDrill, symbol CONN_01X08
- added P3: OLED_0.96in_SPI, library:SolderWirePad_Circle_7xInline_0-85mmDrill, symbol OLED_0.96in_SPI
- added U4: CP2102_Module, library:CP2102Module, symbol CP2102_Module
- added U5: GY-LSM6DS3Module, library:GY-LSM6DS3Module, symbol GY-LSM6DS3Module
- C1, C3, C4: footprint library:C_1206_HandSoldering_Small -> Capacitors_SMD:C_0603
- D1: footprint Diodes_SMD:MELF_Standard -> Diodes_SMD:TUMD2
Connections:
- net +3V3: now also P3.2 (VCC), U4.1 (3V3), U5.2 (3V3)
- net GND: now also P3.1 (GND), U4.2 (GND), U5.3 (GND); no longer BT1.2
- net at U2.29 (P0.27): now also U4.5 (RXD)
- net at U2.30 (P0.25): now also SW1.2, U2.8 (P0.17)
- net at SP1.1, U2.22 (P0.04/AIN2): now also P2.3 (P3)
- net at BT1.1, U6.3 (OUT+), U7.1 (CONTROL)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: now also U6.4 (BAT+), U5.1 (VIN); no longer D1.1 (K)
- net at U2.12 (P0.10/NFC2): now also P2.7 (P7)
- net at U2.13 (P0.09/NFC1): now also P2.6 (P6)
- net at U2.16 (P0.08): now also U5.7 (SA0)
- net at U2.17 (P0.06): now also U5.6 (CS)
- net at U2.18 (P0.07), U8.1 (~CS): now also P2.5 (P5)
- net at U2.19 (P0.05/AIN3): now also P2.4 (P4)
- net at U2.2 (P0.23), U8.5 (MOSI): now also P3.4 (D1)
- net at U2.20 (P0.00/XL1): now also U5.4 (SCL)
- net at U2.21 (P0.01/XL2): now also P2.1 (P1), P3.7 (CS)
- net at U2.23 (P0.03/AIN1), U3.2 (DIN): now also P2.2 (P2)
- net at U2.24 (P0.02/AIN0): now also P3.5 (RST)
- net at U2.3 (P0.22), U8.6 (SCK): now also P3.3 (D0)
- net at U2.31 (P0.30/AIN6): now also U5.5 (SDA)
- net at U2.34 (P0.11): now also P2.8 (P8)
- net at U2.6 (P0.21/RESET), U8.2 (MISO): now also P3.6 (DC)
- net at U6.5 (BAT-): now also BT1.2, D1.2 (A)
- net at P4.1 (P1): now also D1.1 (K); no longer D1.2 (A)
- net +5V: no longer names the net of U6.1 (IN+)
- net +5V: now also U4.3 (+5V)
- new net: U2.35 (P0.26), U4.4 (TXD)
- no-connect marks 44 -> 31
Other:
- note added: "BreadBoard\n"
- note added: "I2C"
- note added: "SCK MOSI RESET \nMISO/DATA \nChipSelect"
- note added: "ST-Link\n"
- note removed: "GND\n3.3V\n5V\nRX\nTX"
- note removed: "MISO MOSI"
- note removed: "SCL SDA SCK"
- moved on the sheet: BT1, C2, C4, D1, P4, U1, U7
