File: KiCad/_autosave-MDBT42STICK.kicad_pcb (KiCad board)
At the start: 2 copper layers, 66 x 32.2 mm, 26 parts, among them P1 CONN_01X04, P12 SERIALBUS, P2 USB_B, P3 CONN_01X07, P4 CONN_01X01, SW1 RESET, U1 ADMP401Module, U2 MDBT42, U3 addressableLEDchip, U5 MPU-6500_Module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

Commit message: 2nd version.
Parts:
- removed the C1 at (76.6, 78.7)
- removed P12: SERIALBUS, library:SolderWirePad_Circle_5xInline_0-8mmDrill
- removed the P2 at (126.2, 67.4)
- removed the P2 at (116.2, 81.9)
- removed the SP1 at (73.0, 65.7)
- removed SW1: RESET, Pin_Headers:Pin_Header_Straight_1x02
- removed U3 (x2): addressableLEDchip, library:addressableLEDchip3535
- removed U5 (x2): MPU-6500_Module, library:MPU-6500_GY-6500
- removed the U6 at (137.9, 87.3)
- removed the U6 at (105.5, 81.9)
- removed the U8 at (75.1, 97.9)
- added ?: GY-LSM6DS3Module, library:GY-LSM6DS3Module, F.Cu at (61.0, 82.5)
- added ?: OLED_0.96in_SPI, library:SolderWirePad_Circle_7xInline_0-85mmDrill, F.Cu at (61.0, 77.4)
- added C1: 0.1uF, Capacitors_SMD:C_0603, F.Cu at (78.2, 79.3)
- added C1: 0.1, Capacitors_SMD:C_0603, F.Cu at (4.79, 74.9)
- added C2: 10, Capacitors_SMD:C_0603, F.Cu at (4.79, 88.5)
- added OSHW: 1.1, library:OSHW_LOGL_SYLK_5mm, F.Cu at (127.7, 82.5)
- added OSHW: 1.1, library:OSHW_LOGL_SYLK_5mm, F.Cu at (139.1, 82.7)
- added OSHW: 1.1, library:OSHW_LOGL_SYLK_5mm, F.Cu at (-6.41, 81.7)
- added P1: CONN_01X10, Connectors_Molex:Connector_Molex_PicoBlade_53047-1010, F.Cu at (-0.41, 75.7)
- added P2: , library:SolderWirePad_Circle_8xInline_0-85mmDrill, F.Cu at (80.1, 87.6)
- added P2: CONN_01X05, Connectors_Molex:Connector_Molex_PicoBlade_53047-0510, F.Cu at (10.2, 89.9)
- added R1: 4.7k, Resistors_SMD:R_0603, F.Cu at (12.2, 72.9)
- added R2: 4.7k, Resistors_SMD:R_0603, F.Cu at (12.2, 75.1)
- added R3: 1.8k, Resistors_SMD:R_0603, F.Cu at (15.8, 72.9)
- added R4: 1.8k, Resistors_SMD:R_0603, F.Cu at (15.8, 75.1)
- added R5: 20k, Resistors_SMD:R_0603, F.Cu at (6.39, 90.7)
- added REF**: SolderWirePad_single_1-2mmDrill, Wire_Pads:SolderWirePad_single_1-2mmDrill, F.Cu at (26.1, 81.9)
- added U4: CP2102_Module, library:CP2102Module, F.Cu at (40.4, 82.2)
- added U6: TP4056Module, library:TP4056Module, F.Cu at (36.6, 82.2)
- ?: renamed from P4; value CONN_01X01 -> (none)
- C3, C4: footprint library:C_1206_HandSoldering_Small -> Capacitors_SMD:C_0603
- D1: footprint Diodes_SMD:MELF_Standard -> Diodes_SMD:TUMD2
- P1: value CONN_01X04 -> (none)
- P3: value CONN_01X07 -> CONN_01X04; footprint Pin_Headers:Pin_Header_Straight_1x07 -> library:Grove_I2C_Horisontal_4pin_2mmpitch
- U1: value ADMP401Module -> MTCH6102_SSOP28; footprint library:ADMP401_Module -> Housings_SSOP:TSSOP-28_4.4x9.7mm_Pitch0.65mm
- moved U1 97.8 mm to (6.59, 81.7), turned to 180 degrees
- moved P3 74.7 mm to (13.6, 81.7), turned to 90 degrees
- moved BT1 52.1 mm to (53.4, 85.1)
- moved C3 47.5 mm to (59.3, 79.9)
- moved ? 41.1 mm to (54.4, 81.7), turned to 90 degrees
- moved U1 25.4 mm to (73.7, 82.5), turned to 270 degrees
- moved C4 20.8 mm to (75.1, 79.3), turned to 0 degrees
- moved P1 10.4 mm to (71.2, 77.4)
- moved SP1 9.03 mm to (64.6, 83.2), turned to 90 degrees
- moved ? 7.73 mm to (59.1, 82.5)
- moved D1 6.02 mm to (58.8, 85.7)
- moved U8 1.80 mm to (75.0, 83.1)
- moved U2 1.37 mm to (87.0, 81.2)
- renumbered U7 to ?
Connections:
- ? pad 1: Net-(D1-Pad2) -> Net-(D1-Pad1)
- BT1 pad 2: GND -> Net-(BT1-Pad2)
- D1 pad 1: Net-(BT1-Pad1) -> Net-(D1-Pad1)
- D1 pad 2: Net-(D1-Pad2) -> Net-(BT1-Pad2)
- P3 pad 1: +3V3 -> Net-(C1-Pad2)
- P3 pad 2: GND -> Net-(C1-Pad1)
- SP1 pad 1: Net-(SP1-Pad1) -> Net-(P2-Pad3)
- U1 pad 1: Net-(U1-Pad1) -> Net-(R5-Pad2)
- U1 pad 2: GND -> Net-(P1-Pad10)
- U1 pad 3: +3V3 -> Net-(P2-Pad1)
- U2 pad 18: Net-(U2-Pad18) -> Net-(P2-Pad5)
- U2 pad 19: Net-(U2-Pad19) -> Net-(P2-Pad4)
- U2 pad 2: Net-(P3-Pad7) -> Net-(P3-Pad4)
- U2 pad 21: Net-(P3-Pad3) -> Net-(P2-Pad1)
- U2 pad 22: Net-(SP1-Pad1) -> Net-(P2-Pad3)
- U2 pad 23: Net-(U2-Pad23) -> Net-(P2-Pad2)
- U2 pad 24: Net-(P3-Pad4) -> Net-(P3-Pad5)
- U2 pad 3: Net-(P3-Pad6) -> Net-(P3-Pad3)
- U2 pad 30: Net-(P12-Pad2) -> Net-(SW1-Pad2)
- U2 pad 35: Net-(SW1-Pad2) -> Net-(U2-Pad35)
- U2 pad 6: Net-(P3-Pad5) -> Net-(P3-Pad6)
- U8 pad 1: Net-(U2-Pad18) -> Net-(P2-Pad5)
- U8 pad 2: Net-(P3-Pad5) -> Net-(P3-Pad6)
- U8 pad 5: Net-(P3-Pad7) -> Net-(P3-Pad4)
- U8 pad 6: Net-(P3-Pad6) -> Net-(P3-Pad3)
Routing:
- net (no net): track 0.00 -> 753.1 mm, vias 0 -> 41
- net GND: track 174.0 -> 32.1 mm, vias 5 -> 2
- net +3V3: track 113.0 -> 0.75 mm, vias 6 -> 0
- net Net-(C1-Pad1): track 0.00 -> 44.9 mm, vias 0 -> 2
- net Net-(BT1-Pad1): track 57.5 -> 13.0 mm, vias 1 -> 0
- net Net-(U1-Pad1): track 38.4 -> 0.00 mm, vias 2 -> 0
- net Net-(SW1-Pad2): track 35.9 -> 0.00 mm, vias 4 -> 0
- net Net-(C1-Pad2): track 0.00 -> 34.6 mm
- net Net-(U2-Pad23): track 33.4 -> 0.00 mm, vias 4 -> 0
- net Net-(U2-Pad31): track 32.5 -> 0.00 mm
- net Net-(P3-Pad7): track 29.7 -> 0.00 mm, vias 2 -> 0
- net Net-(P3-Pad6): track 29.0 -> 0.00 mm, vias 2 -> 0
- net Net-(P12-Pad2): track 19.7 -> 0.00 mm, vias 1 -> 0
- net Net-(P3-Pad5): track 20.3 -> 1.36 mm, vias 2 -> 0
- net Net-(U2-Pad29): track 16.5 -> 0.00 mm, vias 1 -> 0
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Other:
- board size 66 x 32.2 mm -> 159 x 31 mm
- board text added: "00SCL 03SDA 06CS 08SA0"
- board text added: "01 03A1 04A2 05A3 07 09 10 11"
- board text added: "3V3 GND"
- board text added: "3V3 GND +5V ▲RX ▼TX DTR"
- board text added: "3V3 GND +5V ▼RX ▲TX DTR"
- board text added: "B+ B-"
- board text added: "CLK 3V3 DIO GND"
- board text added: "GND SIO 3.3 CLK"
- board text added: "MISO MOSI"
- board text added: "SCL MISO RST MOSI SCK"
- board text added: "SPI OLED Module"
- board text added: "ST-Link"
- board text added: "VIN 3V3 GND"
- board text added: "▼31A7"
- board text added: "▼Breadboard"
- board text added: "▼GYLOModule"
- board text added: "▼Speaker"
- board text removed: "+ - BATT"
- board text removed: "GND 3V3 5NC RX TX"
- board text removed: "GND CLK 3.3 SIO"
